Commit message: updated urdf and meshes

File: robot_control/urdf/surgical_robot.urdf (robot description, URDF)
Before this commit: robot surgical_robot, 3 links, 2 joints
Links:
- link base_link: geometry visual box size=4 4 1
- link pan_link: geometry visual mesh filename=package://robot_control/meshes/Ellipse.dae
- link tilt_link: geometry visual cylinder length=2 radius=0.5
Joints:
- removed joint joint_base_pan
- removed joint joint_shoulder_tilt
- added joint pan_joint: type revolute, parent base_link, child pan_link, origin xyz=0 0 0.5 rpy=0 0 0, axis 0 0 1, limit lower=-3.14 upper=3.14 effort=30 velocity=1.0
- added joint tilt_joint: type revolute, parent pan_link, child tilt_link, origin xyz=0 0 6 rpy=0 0 0, axis 0 1 0, limit lower=-1.57 upper=1.57 effort=30 velocity=1.0
